Commit message: Update allegro_hand_r.urdf

File: src/allegro_hand_model/urdf/allegro_hand_r.urdf (robot description, URDF)
Before this commit: robot allegro_hand_r, 21 links, 20 joints
Links:
- link base_link: mass 4.1685782e+02 -> 0.0041685782e+0.002
- link if1: mass 1.1350110e+01 -> 0.0011350110e+0.001
- link if2: mass None -> 0.0071189096e+0.001
- link if3: mass 3.7588606e+01 -> 0.0037588606e+0.001
- link if4: mass 9.4301124e+00 -> 0.0094301124e+00
- link if5: mass 1.6654268e+01 -> 0.0016654268e+0.001
- link mf1: mass 1.1350110e+01 -> 0.0011350110e+0.001
- link mf2: mass 7.1189096e+01 -> 0.0071189096e+0.001
- link mf3: mass 3.7588606e+01 -> 0.0037588606e+0.001
- link mf4: mass 9.4301124e+00 -> 0.0094301124e+00
- link mf5: mass 1.6654268e+01 -> 0.0016654268e+0.001
- link pf1: mass 1.1350110e+01 -> 0.0011350110e+0.001
- link pf2: mass None -> 0.0071189096e+0.001
- link pf3: mass 3.7588606e+01 -> 0.0037588606e+0.001
- link pf4: mass 9.4301124e+00 -> 0.0094301124e+00
- link pf5: mass 1.6654268e+01 -> 0.0016654268e+0.001
- link th1: mass 7.9809876e-02 -> 0.0079809876e-0.002
- link th2: mass 1.1350110e-02 -> 0.0011350110e-0.002
- link th3: mass  4.0206693e-02 ->  0.0040206693e-0.002
- link th4: mass  4.0750131e-02 ->  0.0040750131e-0.002
- link th5: mass 1.6654268e+01 -> 0.0016654268e+0.001

Commit message: added scale 0.001 into inertia

File: src/allegro_hand_model/urdf/allegro_hand_r.urdf (robot description, URDF)
Before this commit: robot allegro_hand_r, 21 links, 20 joints
Links:
- link base_link: mass 0.0041685782e+0.002 -> 4.1685782e+02
- link if1: mass 0.0011350110e+0.001 -> 1.1350110e+01
- link if2: mass 0.0071189096e+0.001 -> 7.1189096e+01
- link if3: mass 0.0037588606e+0.001 -> 3.7588606e+01
- link if4: mass 0.0094301124e+00 -> 9.4301124e+00
- link if5: mass 0.0016654268e+0.001 -> 1.6654268e+01
- link mf1: mass 0.0011350110e+0.001 -> 1.1350110e+01
- link mf2: mass 0.0071189096e+0.001 -> 7.1189096e+01
- link mf3: mass 0.0037588606e+0.001 -> 3.7588606e+01
- link mf4: mass 0.0094301124e+00 -> 9.4301124e+00
- link mf5: mass 0.0016654268e+0.001 -> 1.6654268e+01
- link pf1: mass 0.0011350110e+0.001 -> 1.1350110e+01
- link pf2: mass 0.0071189096e+0.001 -> 7.1189096e+01
- link pf3: mass 0.0037588606e+0.001 -> 3.7588606e+01
- link pf4: mass 0.0094301124e+00 -> 9.4301124e+00
- link pf5: mass 0.0016654268e+0.001 -> 1.6654268e+01
- link th1: mass 0.0079809876e-0.002 -> 7.9809876e-02
- link th2: mass 0.0011350110e-0.002 -> 1.1350110e-02
- link th3: mass  0.0040206693e-0.002 ->  4.0206693e-02
- link th4: mass  0.0040750131e-0.002 ->  4.0750131e-02
- link th5: mass 0.0016654268e+0.001 -> 1.6654268e+01

Commit message: Update allegro_hand_r.urdf
changed joint name
changed mf1 position and jmf2 joint position

File: src/allegro_hand_model/urdf/allegro_hand_r.urdf (robot description, URDF)
Before this commit: robot allegro_hand, 21 links, 20 joints
Joints:
- removed joint if1
- removed joint if2
- removed joint if3
- removed joint if4
- removed joint if5
- removed joint mf1
- removed joint mf2
- removed joint mf3
- removed joint mf4
- removed joint mf5
- removed joint pf1
- removed joint pf2
- removed joint pf3
- removed joint pf4
- removed joint pf5
- removed joint th1
- removed joint th2
- removed joint th3
- removed joint th4
- removed joint th5
- added joint jif1: type revolute, parent base_link, child if1, origin xyz=0 0.045098 0.014293  rpy=-0.0872665 0 0, axis 0 0 1, limit lower=-0.57 upper=0.57 effort=10 velocity=3
- added joint jif2: type revolute, parent if1, child if2, origin xyz=0 0 0  rpy=0 0 0, axis 0 1 0, limit lower=-0.296 upper=1.71 effort=10 velocity=3
- added joint jif3: type revolute, parent if2, child if3, origin xyz=0 0 0.054 rpy=0 -1.5708 0, axis 0 1 0, limit lower=-0.274 upper=1.809 effort=10 velocity=3
- added joint jif4: type revolute, parent if3, child if4, origin xyz=0.0384 0 0, axis 0 1 0, limit lower=-0.327 upper=1.718 effort=10 velocity=3
- added joint jif5: type fixed, parent if4, child if5, origin xyz=0.0157 0 0
- added joint jmf1: type revolute, parent base_link, child mf1, origin xyz=0 0 0.0166 , axis 0 0 1, limit lower=-0.57 upper=0.57 effort=10 velocity=3
- added joint jmf2: type revolute, parent mf1, child mf2, origin xyz=0 0 0, axis 0 1 0, limit lower=-0.296 upper= 1.71 effort=10 velocity=3
- added joint jmf3: type revolute, parent mf2, child mf3, origin xyz=0 0 0.054 rpy=0 -1.5708 0, axis 0 1 0, limit lower=-0.274 upper= 1.809 effort=10 velocity=3
- added joint jmf4: type revolute, parent mf3, child mf4, origin xyz=0.0384 0 0 rpy=0 0 0, axis 0 1 0, limit lower=-0.327 upper=1.718 effort=10 velocity=3
- added joint jmf5: type fixed, parent mf4, child mf5, origin xyz=0.0157 0 0
- added joint jpf1: type revolute, parent base_link, child pf1, origin xyz=0 -0.045098 0.014293  rpy=0.0872665 0 0, axis 0 0 1, limit lower=-0.57 upper=0.57 effort=10 velocity=3
- added joint jpf2: type revolute, parent pf1, child pf2, origin xyz=0 0 0  rpy=0 0 0, axis 0 1 0, limit lower=-0.296 upper=1.71 effort=10 velocity=3
- added joint jpf3: type revolute, parent pf2, child pf3, origin xyz=0 0 0.054 rpy=0 -1.5708 0, axis 0 1 0, limit lower=-0.274 upper=1.809 effort=10 velocity=3
- added joint jpf4: type revolute, parent pf3, child pf4, origin xyz=0.0384 0 0, axis 0 1 0, limit lower=-0.327 upper=1.718 effort=10 velocity=3
- added joint jpf5: type fixed, parent pf4, child pf5, origin xyz=0.0157 0 0
- added joint jth1: type revolute, parent base_link, child th1, origin xyz=-0.0182 0.016958 -0.073288  rpy=-0.0872665 0 0, axis 0 0 -1, limit lower=0.36357 upper=1.4968 effort=10 velocity=3
- added joint jth2: type revolute, parent th1, child th2, origin xyz=0.005 0.055189 0  rpy=0 0 0, axis 0 1 0, limit lower=-0.20504289 upper=1.263 effort=10 velocity=3
- added joint jth3: type revolute, parent th2, child th3, origin xyz=0 0 0  rpy=0 0 0, axis 1 0 0, limit lower=-0.2897 upper=1.7440 effort=10 velocity=3
- added joint jth4: type revolute, parent th3, child th4, origin xyz=0 0.051204 0  rpy=0 0 0, axis 1 0 0, limit lower=-0.2622 upper=1.81991 effort=10 velocity=3
- added joint jth5: type fixed, parent th4, child th5, origin xyz=0 0.0313 0  rpy=0 -1.4835335 0

Commit message: Fixed th1 collision issue,etc

File: src/allegro_hand_model/urdf/allegro_hand_r.urdf (robot description, URDF)
Before this commit: robot allegro_hand, 21 links, 20 joints
Links:
- link th1: geometry collision mesh filename=package://allegro_hand_model/meshes/40_10_link_t1_r.stl scale=0.001 0.001 0.001; visual mesh filename=package://allegro_hand_model/meshes/40_10_link_t1_r.stl scale=0.001 0.001 0.001
Joints:
- joint jth1: origin xyz=-0.0182 0.016958 -0.073288  rpy=-0.0872665 0 0 -> xyz=-0.0182 0.016958 -0.0723  rpy=-0.0872665 0 0

Commit message: fixed collision scale and issue

File: src/allegro_hand_model/urdf/allegro_hand_r.urdf (robot description, URDF)
Before this commit: robot allegro_hand, 21 links, 20 joints
Links:
- link th3: geometry collision mesh filename=package://allegro_hand_model/meshes/40_10_link_t3.stl scale=0.001 0.001 0.001; visual mesh filename=package://allegro_hand_model/meshes/40_10_link_t3.stl scale=0.001 0.001 0.001
- link th4: geometry collision mesh filename=package://allegro_hand_model/meshes/40_10_link_t4.stl scale=0.001 0.001 0.001; visual mesh filename=package://allegro_hand_model/meshes/40_10_link_t4.stl scale=0.001 0.001 0.001
Joints:
- joint jth3: limit lower=-0.2897 upper=1.7440 effort=10 velocity=3 -> lower=-0.2897 upper=1.633 effort=10 velocity=3
- joint jth4: origin xyz=0 0.051204 0  rpy=0 0 0 -> xyz=0 0.051204 -0.00448  rpy=0 0 0

Commit message: fixed th4 issue and joint scale to prevent colli

File: src/allegro_hand_model/urdf/allegro_hand_r.urdf (robot description, URDF)
Before this commit: robot allegro_hand, 21 links, 20 joints
Joints:
- joint jth2: limit lower=-0.20504289 upper=1.263 effort=10 velocity=3 -> lower=-0.20504289 upper=1.13 effort=10 velocity=3
- joint jth4: origin xyz=0 0.051204 -0.00448  rpy=0 0 0 -> xyz=0 0.051204 0  rpy=0 0 0

Commit message: fixed mass and model of th2

File: src/allegro_hand_model/urdf/allegro_hand_r.urdf (robot description, URDF)
Before this commit: robot allegro_hand, 21 links, 20 joints
Links:
- link th2: mass 1.1350110e-02 -> 1.1350110e+01; geometry collision mesh filename=package://allegro_hand_model/meshes/40_10_link_f1.stl; visual mesh filename=package://allegro_hand_model/meshes/40_10_link_f1.stl

Commit message: changed to none bearing model, inertia scale

File: src/allegro_hand_model/urdf/allegro_hand_r.urdf (robot description, URDF)
Before this commit: robot allegro_hand, 21 links, 20 joints
Links:
- link base_link: geometry collision mesh filename=package://allegro_hand_model/meshes/40_10_link_g_r.stl scale=0.001 0.001 0.001; visual mesh filename=package://allegro_hand_model/meshes/40_10_link_g_r.stl scale=0.001 0.001 0.001
- link if1: geometry collision mesh filename=package://allegro_hand_model/meshes/40_10_link_f1.stl scale=0.001 0.001 0.001; visual mesh filename=package://allegro_hand_model/meshes/40_10_link_f1.stl scale=0.001 0.001 0.001
- link if2: geometry collision mesh filename=package://allegro_hand_model/meshes/40_10_link_f2.stl scale=0.001 0.001 0.001; visual mesh filename=package://allegro_hand_model/meshes/40_10_link_f2.stl scale=0.001 0.001 0.001
- link if3: geometry collision mesh filename=package://allegro_hand_model/meshes/40_10_link_f3.stl scale=0.001 0.001 0.001; visual mesh filename=package://allegro_hand_model/meshes/40_10_link_f3.stl scale=0.001 0.001 0.001
- link if4: geometry collision mesh filename=package://allegro_hand_model/meshes/40_10_link_f4.stl scale=0.001 0.001 0.001; visual mesh filename=package://allegro_hand_model/meshes/40_10_link_f4.stl scale=0.001 0.001 0.001
- link if5: geometry collision mesh filename=package://allegro_hand_model/meshes/40_10_link_f5.stl scale=0.001 0.001 0.001; visual mesh filename=package://allegro_hand_model/meshes/40_10_link_f5.stl scale=0.001 0.001 0.001
- link mf1: geometry collision mesh filename=package://allegro_hand_model/meshes/40_10_link_f1.stl scale=0.001 0.001 0.001; visual mesh filename=package://allegro_hand_model/meshes/40_10_link_f1.stl scale=0.001 0.001 0.001
- link mf2: geometry collision mesh filename=package://allegro_hand_model/meshes/40_10_link_f2.stl scale=0.001 0.001 0.001; visual mesh filename=package://allegro_hand_model/meshes/40_10_link_f2.stl scale=0.001 0.001 0.001
- link mf3: geometry collision mesh filename=package://allegro_hand_model/meshes/40_10_link_f3.stl scale=0.001 0.001 0.001; visual mesh filename=package://allegro_hand_model/meshes/40_10_link_f3.stl scale=0.001 0.001 0.001
- link mf4: geometry collision mesh filename=package://allegro_hand_model/meshes/40_10_link_f4.stl scale=0.001 0.001 0.001; visual mesh filename=package://allegro_hand_model/meshes/40_10_link_f4.stl scale=0.001 0.001 0.001
- link mf5: geometry collision mesh filename=package://allegro_hand_model/meshes/40_10_link_f5.stl scale=0.001 0.001 0.001; visual mesh filename=package://allegro_hand_model/meshes/40_10_link_f5.stl scale=0.001 0.001 0.001
- link pf1: geometry collision mesh filename=package://allegro_hand_model/meshes/40_10_link_f1.stl scale=0.001 0.001 0.001; visual mesh filename=package://allegro_hand_model/meshes/40_10_link_f1.stl scale=0.001 0.001 0.001
- link pf2: geometry collision mesh filename=package://allegro_hand_model/meshes/40_10_link_f2.stl scale=0.001 0.001 0.001; visual mesh filename=package://allegro_hand_model/meshes/40_10_link_f2.stl scale=0.001 0.001 0.001
- link pf3: geometry collision mesh filename=package://allegro_hand_model/meshes/40_10_link_f3.stl scale=0.001 0.001 0.001; visual mesh filename=package://allegro_hand_model/meshes/40_10_link_f3.stl scale=0.001 0.001 0.001
- link pf4: geometry collision mesh filename=package://allegro_hand_model/meshes/40_10_link_f4.stl scale=0.001 0.001 0.001; visual mesh filename=package://allegro_hand_model/meshes/40_10_link_f4.stl scale=0.001 0.001 0.001
- link pf5: geometry collision mesh filename=package://allegro_hand_model/meshes/40_10_link_f5.stl scale=0.001 0.001 0.001; visual mesh filename=package://allegro_hand_model/meshes/40_10_link_f5.stl scale=0.001 0.001 0.001
- link th2: geometry collision mesh filename=package://allegro_hand_model/meshes/40_10_link_f1.stl scale=0.001 0.001 0.001; visual mesh filename=package://allegro_hand_model/meshes/40_10_link_f1.stl scale=0.001 0.001 0.001
- link th5: geometry collision mesh filename=package://allegro_hand_model/meshes/40_10_link_f5.stl scale=0.001 0.001 0.001; visual mesh filename=package://allegro_hand_model/meshes/40_10_link_f5.stl scale=0.001 0.001 0.001

Commit message: changed inertia and mass to right data

File: src/allegro_hand_model/urdf/allegro_hand_r.urdf (robot description, URDF)
Before this commit: robot allegro_hand, 21 links, 20 joints
Links:
- link base_link: mass 4.1685782e+02 -> 4.1685782e-01
- link if1: mass 1.1350110e+01 -> 1.1350110e-02
- link if2: mass 7.1189096e+01 -> 7.1189096e-02
- link if3: mass 3.7588606e+01 -> 3.7588606e-02
- link if4: mass 9.4301124e+00 -> 9.4301124e-03
- link if5: mass 1.6654268e+01 -> 1.6654268e-02
- link mf1: mass 1.1350110e+01 -> 1.1350110e-02
- link mf2: mass 7.1189096e+01 -> 7.1189096e-02
- link mf3: mass 3.7588606e+01 -> 3.7588606e-02
- link mf4: mass 9.4301124e+00 -> 9.4301124e-03
- link mf5: mass 1.6654268e+01 -> 1.6654268e-02
- link pf1: mass 1.1350110e+01 -> 1.1350110e-02
- link pf2: mass 7.1189096e+01 -> 7.1189096e-02
- link pf3: mass 3.7588606e+01 -> 3.7588606e-02
- link pf4: mass 9.4301124e+00 -> 9.4301124e-03
- link pf5: mass 1.6654268e+01 -> 1.6654268e-02
- link th2: mass 1.1350110e+01 -> 1.1350110e-02
- link th5: mass 1.6654268e+01 -> 1.6654268e-02

Commit message: changed inertia

File: src/allegro_hand_model/urdf/allegro_hand_r.urdf (robot description, URDF)
Before this commit: robot allegro_hand, 21 links, 20 joints
Links:
- link th3: mass  4.0206693e-02 -> 4.0206693e-02
